File: eeprom-sync/vga/vga/vga.kicad_sch (KiCad schematic)
At the start: 1 part

Commit message: schematic updated
Parts:
- added R? (x12): 680, symbol Device:R_US
- added R? (x6): 330, symbol Device:R_US
- added U?: 74HC273, symbol 74xx:74HC273
- added U? (x3): 74LS04, symbol 74xx:74LS04
- added U?: 74LS32, symbol 74xx:74LS32
- added U? (x2): IDT7204, Package_DIP:DIP-28_W7.62mm, symbol Memory_RAM:IDT7204
- added U?: GAL22V10, symbol vga:GAL22V10
Connections:
- net Earth: now reaches U?.12 (GND)
- net Earth: now also R?.1, R?.1, R?.1, U?.10 (GND), U?.12 (GND), U?.14 (GND), U?.14 (GND), U?.23 (~{FL}/~{RT})
- net at U?.23 (IO1): now also U?.1 (~{W}), U?.1 (~{W})
- net +5V: now reaches U?.24 (VCC)
- net +5V: now also U?.1 (~{Mr}), U?.20 (VCC), U?.23 (~{FL}/~{RT}), U?.24 (VCC), U?.28 (VCC), U?.28 (VCC)
- new net: U?.11 (Cp), U?.2
- new net: R?.2, R?.2, R?.2 (x3)
- new net: U?.1, U?.15 (~{R}), U?.15 (~{R}), U?.3
- new net: U?.1, U?.2
- new net: R?.1, R?.1, R?.2 (x3)
- new net: U?.20 (~{HF}/~{XO}), U?.7 (~{XI}) (x2)
- new net: U?.2, U?.22 (~{RS}), U?.22 (~{RS})
- new net Blue: R?.2, R?.2
- new net Frame_Vis: U?.11 (I11)
- new net GPIO3: U?.1
- new net Not_Frame_Vis: U?.2
- new net Pixel_Clock: U?.1
- new net Red: R?.2, R?.2, R?.2, R?.2
Other:
- note added: "SIPO"

Commit message: vga schematic and pcb layout
Parts:
- removed U? (x2): 74LS04, symbol 74xx:74LS04
- added J1: Conn_01x02_Male, Connector_PinHeader_2.54mm:PinHeader_1x02_P2.54mm_Vertical, symbol Connector:Conn_01x02_Male
- added J2: Conn_01x04_Female, Connector_PinSocket_2.54mm:PinSocket_1x04_P2.54mm_Vertical, symbol Connector:Conn_01x04_Female
- added J3, J4: Conn_01x15_Female, Connector_PinSocket_2.54mm:PinSocket_1x15_P2.54mm_Vertical, symbol Connector:Conn_01x15_Female
- added J5: Conn_01x02_Female, Connector_PinSocket_2.54mm:PinSocket_1x02_P2.54mm_Vertical, symbol Connector:Conn_01x02_Female
- added J6: DB15_Female_HighDensity_MountingHoles, Connector_Dsub:DSUB-15_Female_Horizontal_P2.77x2.84mm_EdgePinOffset4.94mm_Housed_MountingHolesOffset7.48mm, symbol Connector:DB15_Female_HighDensity_MountingHoles
- added U10, U12, U14, U15, U6: 74LS163 (! HC?), Package_DIP:DIP-16_W7.62mm, symbol 74xx:74LS163
- added U11: 28C256, Package_DIP:DIP-28_W15.24mm_Socket, symbol Memory_EEPROM:28C256
- added U13: 74HCT574, Package_DIP:DIP-20_W7.62mm, symbol 74xx:74HCT574
- added unit 3 of U3
- added unit 2 of U3
- added X1: CXO_DIP8, Oscillator:Oscillator_DIP-8, symbol Oscillator:CXO_DIP8
- R1, R10, R11, R12, R13, R14, R15, R16, R17, R18, R2, R3, R4, R5, R6, R7, R8, R9: renamed from R?; footprint (none) -> Resistor_THT:R_Axial_DIN0204_L3.6mm_D1.6mm_P5.08mm_Horizontal
- U1, U9: renamed from U?; footprint (none) -> Package_DIP:DIP-24_W7.62mm_Socket
- U3, U4: renamed from U?; footprint (none) -> Package_DIP:DIP-14_W7.62mm
- U8: renamed from U?; footprint (none) -> Package_DIP:DIP-20_W7.62mm
- gave numbers to parts that had none: 2
Connections:
- net SIO0: now also J3.9 (Pin_9)
- net SIO1: now also J4.4 (Pin_4)
- net SIO2: now also J3.7 (Pin_7)
- net SIO3: now also J3.6 (Pin_6)
- net at U8.11 (Cp): now also U3.6
- net P4: now reaches U8.12 (Q4)
- net P4: now also U9.5 (I5)
- net Q4: now reaches U8.13 (D4)
- net Q4: now also U5.16 (Q4), U7.16 (Q4)
- net Q5: now reaches U8.14 (D5)
- net Q5: now also U5.17 (Q5), U7.17 (Q5)
- net P5: now reaches U8.15 (Q5)
- net P5: now also U9.4 (I4/PD)
- net P6: now reaches U8.16 (Q6)
- net P6: now also U9.3 (I3)
- net Q6: now reaches U8.17 (D6)
- net Q6: now also U5.18 (Q6), U7.18 (Q6)
- net Q7: now reaches U8.18 (D7)
- net Q7: now also U5.19 (Q7), U7.19 (Q7)
- net P7: now reaches U8.19 (Q7)
- net P7: now also U9.2 (I2)
- net P0: now reaches U8.2 (Q0)
- net P0: now also U9.9 (I9)
- net Q0: now reaches U8.3 (D0)
- net Q0: now also U5.9 (Q0), U7.9 (Q0)
- net Q1: now reaches U8.4 (D1)
- net Q1: now also U5.10 (Q1), U7.10 (Q1)
- net P1: now reaches U8.5 (Q1)
- net P1: now also U9.8 (I8)
- net P2: now reaches U8.6 (Q2)
- net P2: now also U9.7 (I7)
- net Q2: now reaches U8.7 (D2)
- net Q2: now also U5.11 (Q2), U7.11 (Q2)
- net Q3: now reaches U8.8 (D3)
- net Q3: now also U5.12 (Q3), U7.12 (Q3)
- net P3: now reaches U8.9 (Q3)
- net P3: now also U9.6 (I6)
- net at U4.3, U5.15 (~{R}), U7.15 (~{R}): now also U3.5
- net Blue1: now reaches R15.1
- net Blue1: now also U9.15 (IO9)
- net Red0: now reaches R5.1
- net Red0: now also U9.22 (IO2)
- net Red1: now reaches R3.1
- net Red1: now also U9.21 (I03)
- net Green1: now reaches R9.1
- net Green1: now also U9.18 (IO6)
- net Green0: now reaches R11.1
- net Green0: now also U9.19 (IO5)
- net at U5.22 (~{RS}), U7.22 (~{RS}): now also U3.4
- net D7: now reaches U5.24 (D7)
- net D7: now also U1.21 (I03), U7.24 (D7)
- net D6: now reaches U5.25 (D6)
- net D6: now also U1.20 (IO4), U7.25 (D6)
- net D5: now reaches U5.26 (D5)
- net D5: now also U1.19 (IO5), U7.26 (D5)
- net D4: now reaches U5.27 (D4)
- net D4: now also U1.18 (IO6), U7.27 (D4)
- net D3: now reaches U5.3 (D3)
- net D3: now also U1.17 (IO7), U7.3 (D3)
- net D2: now reaches U5.4 (D2)
- net D2: now also U1.16 (IO8), U7.4 (D2)
- net D1: now reaches U5.5 (D1)
- net D1: now also U1.15 (IO9), U7.5 (D1)
- net D0: now reaches U5.6 (D0)
- net D0: now also U1.14 (IO10), U7.6 (D0)
- net Blue0: now reaches R17.1
- net Blue0: now also U9.16 (IO8)
- net Blue2: now reaches R13.1
- net Blue2: now also U9.14 (IO10)
- net Red2: now reaches R1.1
- net Red2: now also U9.20 (IO4)
- net Green2: now reaches R7.1
- net Green2: now also U9.17 (IO7)
- net +5V renamed VCC
- net VCC: now also J1.1 (Pin_1), J2.3 (Pin_3), J3.13 (Pin_13), J3.14 (Pin_14), J5.1 (Pin_1), U10.16 (VCC), U10.7 (CEP), U10.9 (~{PE}), U11.27 (~{WE}), U11.28 (VCC), U12.16 (VCC), U12.7 (CEP), U12.9 (~{PE}), U13.20 (VCC), U14.10 (CET), U14.16 (VCC), U14.7 (CEP), U14.9 (~{PE}), U15.1 (~{MR}), U15.10 (CET), U15.16 (VCC), U15.7 (CEP), U6.16 (VCC), U6.7 (CEP), U6.9 (~{PE}), X1.8 (Vcc)
- net Blue renamed G_{out}
- net G_{out}: now also J6.2
- net Earth renamed GND
- net GND: now also J1.2 (Pin_2), J2.4 (Pin_4), J3.1 (Pin_1), J3.10 (Pin_10), J3.15 (Pin_15), J3.5 (Pin_5), J4.1 (Pin_1), J4.11 (Pin_11), J4.14 (Pin_14), J4.15 (Pin_15), J4.6 (Pin_6), J4.8 (Pin_8), J5.2 (Pin_2), J6.0, J6.10, J6.5, U10.8 (GND), U11.14 (GND), U11.20 (~{CS}), U11.22 (~{OE}), U12.8 (GND), U13.1 (OE), U13.10 (GND), U14.8 (GND), U15.8 (GND), U6.8 (GND), X1.4 (GND)
- net Frame_Vis renamed Vis
- net Vis: now also U13.15 (Q4)
- net Not_Frame_Vis renamed ~{Vis}
- net ~{Vis}: now also U13.14 (Q5)
- net Pixel_Clock renamed CLK_{pixel}
- net CLK_{pixel}: now also U15.2 (CP), X1.5 (OUT)
- net Red renamed B_{out}
- net B_{out}: now also J6.3; no longer R1.2, R2.2
- net SPI Clock renamed SCLK
- net SCLK: now also J3.8 (Pin_8)
- new net: U11.11 (D0), U13.2 (D0)
- new net: U11.12 (D1), U13.3 (D1)
- new net: U11.13 (D2), U13.4 (D2)
- new net: U11.15 (D3), U13.5 (D3)
- new net: U11.16 (D4), U13.6 (D4)
- new net: U11.17 (D5), U13.7 (D5)
- new net: U11.18 (D6), U13.8 (D6)
- new net: U10.15 (TC), U6.10 (CET)
- new net: U12.10 (CET), U14.15 (TC)
- new net: U10.10 (CET), U12.15 (TC)
- new net A0: U11.10 (A0), U14.14 (Q0)
- new net A1: U11.9 (A1), U14.13 (Q1)
- new net A10: U10.12 (Q2), U11.21 (A10)
- new net A11: U10.11 (Q3), U11.23 (A11)
- new net A12: U11.2 (A12), U6.14 (Q0)
- new net A13: U11.26 (A13), U6.13 (Q1)
- new net A14: U11.1 (A14), U6.12 (Q2)
- new net A2: U11.8 (A2), U14.12 (Q2)
- new net A3: U11.7 (A3), U14.11 (Q3)
- new net A4: U11.6 (A4), U12.14 (Q0)
- new net A5: U11.5 (A5), U12.13 (Q1)
- new net A6: U11.4 (A6), U12.12 (Q2)
- new net A7: U11.3 (A7), U12.11 (Q3)
- new net A8: U10.14 (Q0), U11.25 (A8)
- new net A9: U10.13 (Q1), U11.24 (A9)
- new net CLK_{sync}: U10.2 (CP), U12.2 (CP), U13.11 (Cp), U14.2 (CP), U15.11 (Q3), U6.2 (CP)
- new net CS: J4.7 (Pin_7)
- new net D+: J4.13 (Pin_13)
- new net D-: J4.12 (Pin_12)
- new net End: U13.12 (Q7)
- new net HSync: J6.13, U13.18 (Q1)
- new net HVis: U13.19 (Q0)
- new net KB_{Rx}: J2.2 (Pin_2), J4.2 (Pin_2)
- new net KB_{Tx}: J2.1 (Pin_1), J4.3 (Pin_3)
- new net R_{out}: J6.1, R1.2, R2.2
- new net StartFrame: J4.5 (Pin_5), U13.13 (Q6), U3.3
- new net VertVis: U13.17 (Q2)
- new net Vsync: J6.14, U13.16 (Q3)
- new net ~{RESET}: U10.1 (~{MR}), U11.19 (D7), U12.1 (~{MR}), U14.1 (~{MR}), U6.1 (~{MR})
- no-connect marks 0 -> 63
Other:
- moved on the sheet: R1, R10, R11, R12, R13, R14, R15, R16, R17, R18, R2, R3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
