File: eeprom-sync/vga/vga/timing/timing/timing.kicad_sch (KiCad schematic)
At the start: 12 parts, among them J1 Conn_01x02_Male, J2 Conn_01x02_Female, J3 Conn_01x08_Female, U1 74LS161, U2 74LS161, U3 28C256, U4 74LS161, U5 74HCT574, U6 74LS161, U7 74LS08, U8 74LS161, X1 CXO_DIP8

Commit message: final board
Parts:
- removed J3: Conn_01x08_Female, Connector_PinSocket_2.54mm:PinSocket_1x08_P2.54mm_Vertical, symbol Connector:Conn_01x08_Female
- removed U7: 74LS08, Package_SO:TSSOP-14_4.4x5mm_P0.65mm, symbol 74xx:74LS08
- removed X1: CXO_DIP8, Oscillator:Oscillator_DIP-8, symbol Oscillator:CXO_DIP8
- added C1, C2, C3, C4, C5, C6, C7, C8: C_Small, Capacitor_SMD:C_0805_2012Metric_Pad1.18x1.45mm_HandSolder, symbol Device:C_Small
- added J4: Conn_01x09_Socket, Connector_PinSocket_2.54mm:PinSocket_1x09_P2.54mm_Vertical, symbol Connector:Conn_01x09_Socket
- U5: footprint Package_SO:TSSOP-20_4.4x6.5mm_P0.65mm -> Package_SO:SOIC-20W_7.5x12.8mm_P1.27mm
Connections:
- net GND: now also U1.3 (D0), U1.4 (D1), U1.5 (D2), U1.6 (D3), U2.3 (D0), U2.4 (D1), U2.5 (D2), U2.6 (D3), U4.3 (D0), U4.4 (D1), U4.5 (D2), U4.6 (D3), U5.9 (D7), U6.3 (D0), U6.4 (D1), U6.5 (D2), U6.6 (D3), U8.3 (D0), U8.4 (D1), U8.5 (D2), U8.6 (D3), C1.2, C2.2, C3.2, C4.2, C5.2, C6.2, C7.2, C8.2
- net HSync: now also J4.2 (Pin_2)
- net HVis: now also J4.1 (Pin_1)
- net StartFrame: now also J4.7 (Pin_7)
- net VCC: now also U8.9 (~{PE}), C1.1, C2.1, C3.1, C4.1, C5.1, C6.1, C7.1, C8.1
- net VertVis: now also J4.3 (Pin_3)
- net Vis: now also J4.5 (Pin_5)
- net Vsync: now also J4.4 (Pin_4)
- net ~{Vis}: now also J4.6 (Pin_6)
- net Clk_{in}: now reaches U8.2 (CP)
- net Clk_{in}: now also J4.9 (Pin_9)
- net Othr: now reaches U5.12 (Q7)
- net Othr: now also J4.8 (Pin_8)
- no-connect marks 30 -> 6
